Commit message: Update rbvogui_xl_lift_ur10e.urdf

File: data/rbvogui_xl_lift_ur10e.urdf (robot description, URDF)
Before this commit: robot rbvogui, 41 links, 40 joints
Joints:
- joint robot_arm_base_joint: origin xyz=0 0 0.015 rpy=0 0 0 -> xyz=0 0 0.015 rpy=0 0 2.35619449019
- joint robot_arm_base_link-base_link_inertia: origin xyz=0 0 0 rpy=0 0 3.14159265359 -> xyz=0 0 0 rpy=0 0 0

Commit message: urdf fixes

File: data/rbvogui_xl_lift_ur10e.urdf (robot description, URDF)
Before this commit: robot rbvogui, 41 links, 40 joints
Links:
- link robot_ewellix_lift_base_link: geometry collision mesh filename=package://ewellix_description/meshes/ewellix_lift_base_700m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; visual mesh filename=package://ewellix_description/meshes/ewellix_lift_base_700m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
- link robot_ewellix_lift_top_link: geometry collision mesh filename=package://ewellix_description/meshes/ewellix_lift_top_700mm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; visual mesh filename=package://ewellix_description/meshes/ewellix_lift_top_700mm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
Joints:
- joint robot_ewellix_lift_base_joint: origin xyz=0.207 0.0 0.3 rpy=0 0 0 -> xyz=0.275 0.0 0.3 rpy=0 0 0
- joint robot_ewellix_lift_top_joint: limit lower=0.0 upper=0.9 effort=1000 velocity=0.088 -> lower=0.0 upper=0.7 effort=1000 velocity=0.088; origin xyz=0 0 0.730 rpy=0 0 0 -> xyz=0 0 0.620 rpy=0 0 0

Commit message: Update rbvogui_xl_lift_ur10e.urdf

File: data/rbvogui_xl_lift_ur10e.urdf (robot description, URDF)
Before this commit: robot rbvogui, 41 links, 40 joints
Links:
- link robot_base_link: geometry collision mesh filename=package://rbvogui_description/meshes/bases/rbvogui_chassis.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; visual mesh filename=package://rbvogui_description/meshes/bases/rbvogui_chassis.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

Commit message: Update rbvogui_xl_lift_ur10e.urdf

File: data/rbvogui_xl_lift_ur10e.urdf (robot description, URDF)
Before this commit: robot rbvogui, 41 links, 40 joints
Links:
- removed link robot_zed_base_link
- removed link robot_zed_left_rgb_frame
- removed link robot_zed_left_rgb_optical_frame
- removed link robot_zed_right_rgb_frame
- removed link robot_zed_right_rgb_optical_frame
- added link robot_battery_link, mass 20.0; collision mesh filename=package://rbvogui_description/meshes/bases/rbvogui_xl_batte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; visual mesh filename=package://rbvogui_description/meshes/bases/rbvogui_xl_batte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
- added link robot_chassis_link, mass 25.0; collision mesh filename=package://rbvogui_description/meshes/bases/rbvogui_xl_chass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; visual mesh filename=package://rbvogui_description/meshes/bases/rbvogui_xl_chass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
- added link robot_contactors_link; visual mesh filename=package://rbvogui_description/meshes/bases/rbvogui_contacto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
- added link robot_front_rgbd_camera_depth_frame, mass 0.001
- added link robot_front_rgbd_camera_depth_optical_frame, mass 0.001
- added link robot_front_rgbd_camera_link, mass 0.001; collision mesh filename=package://robotnik_sensors/meshes/orbbec_astra.stl; visual mesh filename=package://robotnik_sensors/meshes/orbbec_astra.stl
- added link robot_front_rgbd_camera_rgb_frame, mass 0.297
- added link robot_front_rgbd_camera_rgb_optical_frame, mass 0.001
- added link robot_gps_link
- added link robot_imu_base_link, mass 0.05; collision box size=0.036 0.037 0.009; visual mesh filename=package://robotnik_sensors/meshes/vectornav_vn100.stl
- added link robot_leds_link; visual mesh filename=package://rbvogui_description/meshes/bases/rbvogui_xl_leds.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
- link robot_base_link: mass 25.0 -> None; geometry 
- link robot_base_logos_link: geometry visual mesh filename=package://rbvogui_description/meshes/bases/rbvogui_logos.stl scale=1.24 1.24 1
- link robot_front_laser_base_link: geometry collision box size=0.106 0.094 0.152; visual mesh filename=package://robotnik_sensors/meshes/sick_microscan3.stl
- link robot_gps_base_link: geometry collision mesh filename=package://robotnik_sensors/meshes/antenna_ANN_MB_mast.stl scale=1.0 1.0 1.0; visual mesh filename=package://robotnik_sensors/meshes/antenna_ANN_MB_mast.stl scale=1.0 1.0 1.0
- link robot_imu_link: mass 0.05 -> None; geometry 
- link robot_rear_laser_base_link: geometry collision box size=0.106 0.094 0.152; visual mesh filename=package://robotnik_sensors/meshes/sick_microscan3.stl
Joints:
- removed joint robot_zed_base_joint
- removed joint robot_zed_rgb_left_joint
- removed joint robot_zed_rgb_left_optical_joint
- removed joint robot_zed_rgb_right_joint
- removed joint robot_zed_rgb_right_optical_joint
- added joint robot_battery_joint: type fixed, parent robot_chassis_link, child robot_battery_link, origin xyz=0 0 0 rpy=0 0 0 
- added joint robot_chassis_joint: type fixed, parent robot_base_link, child robot_chassis_link, origin xyz=0 0 0.23376 rpy=0 0 0
- added joint robot_contactors_joint: type fixed, parent robot_chassis_link, child robot_contactors_link, origin xyz=0.6405 0 0.10264 rpy=0 0 0 
- added joint robot_front_rgbd_camera_depth_joint: type fixed, parent robot_front_rgbd_camera_link, child robot_front_rgbd_camera_depth_frame, origin xyz=0.0 0.0375 0.0150 rpy=0 0 0
- added joint robot_front_rgbd_camera_depth_optical_joint: type fixed, parent robot_front_rgbd_camera_depth_frame, child robot_front_rgbd_camera_depth_optical_frame, origin xyz=0 0 0 rpy=-1.57079632679 0 -1.57079632679
- added joint robot_front_rgbd_camera_joint: type fixed, parent robot_chassis_link, child robot_front_rgbd_camera_link, origin xyz=0.637 0.0 -0.036 rpy=0 0 0
- added joint robot_front_rgbd_camera_rgb_joint: type fixed, parent robot_front_rgbd_camera_link, child robot_front_rgbd_camera_rgb_frame, origin xyz=0.0 0.0125 0.0150 rpy=0.0 0.0 0.0
- added joint robot_front_rgbd_camera_rgb_optical_joint: type fixed, parent robot_front_rgbd_camera_rgb_frame, child robot_front_rgbd_camera_rgb_optical_frame, origin xyz=0.0 0.0 0.0 rpy=-1.57079632679 0 -1.57079632679
- added joint robot_gps_base_joint: type fixed, parent robot_chassis_link, child robot_gps_base_link, origin xyz=-0.472 0.4 0.456 rpy=0 0 0, axis 0 1 0
- added joint robot_imu_base_joint: type fixed, parent robot_chassis_link, child robot_imu_base_link, origin xyz=0.3 -0.3 0.0725 rpy=0 0 0, axis 1 0 0
- added joint robot_leds_joint: type fixed, parent robot_chassis_link, child robot_leds_link, origin xyz=0 0 0.12624 rpy=0 0 0 
- joint robot_base_logos_joint: origin xyz=0 0 0.15 rpy=0 0 0  -> xyz=0 0 -0.08376 rpy=0 0 0 ; parent robot_base_link -> robot_chassis_link
- joint robot_ewellix_lift_base_joint: origin xyz=0.275 0.0 0.3 rpy=0 0 0 -> xyz=0.275 0.0 0.01 rpy=0 0 0; parent robot_base_link -> robot_chassis_link
- joint robot_front_3d_laser_base_joint: origin xyz=0.645 0 0.52032 rpy=0 1.57079632679 0 -> xyz=0.579 0 0.241 rpy=0 1.57079632679 0; parent robot_base_link -> robot_chassis_link
- joint robot_front_3d_laser_joint: origin xyz=0 0 0.06 rpy=0 0 0 -> xyz=0 0 0.09427 rpy=0 0 0
- joint robot_front_laser_base_joint: origin xyz=0.645 0.396 0.44559 rpy=3.14159265359 0 0.785398163397 -> xyz=0.64555 0.39595 0.16608 rpy=3.14159265359 0 0.785398163397; parent robot_base_link -> robot_chassis_link
- joint robot_gps_joint: axis 0 1 0 -> 1 0 0; child robot_gps_base_link -> robot_gps_link; origin xyz=-0.04625 0.0 0.59188 rpy=0 0 0 -> xyz=0.0 0.0 0.01125; parent robot_base_link -> robot_gps_base_link
- joint robot_imu_joint: origin xyz=0.3 0.0 0.3 rpy=0 0 0 -> xyz=0.00671 0.0047 0.0059; parent robot_base_link -> robot_imu_base_link
- joint robot_rear_laser_base_joint: origin xyz=-0.645 -0.396 0.44559 rpy=3.14159265359 0 -2.35619449019 -> xyz=-0.64555 -0.39985 0.16608 rpy=3.14159265359 0 -2.35619449019; parent robot_base_link -> robot_chassis_link
- joint robot_sick_front_protectorsick_support_joint: origin xyz=0.645 0.396 0.39025 rpy=0 0 -0.785398163397 -> xyz=0.64542 0.39594 0.11073 rpy=0 0 -0.785398163397; parent robot_base_link -> robot_chassis_link
- joint robot_sick_front_supportsick_support_joint: origin xyz=0.472 0.3795 0.3774 rpy=0 1.57079632679 1.57079632679 -> xyz=0.472 0.3795 0.09788 rpy=0 1.57079632679 1.57079632679; parent robot_base_link -> robot_chassis_link
- joint robot_sick_rear_protectorsick_support_joint: origin xyz=-0.645 -0.396 0.39025 rpy=0 0 2.35619449019 -> xyz=-0.64542 -0.39594 0.11073 rpy=0 0 2.35619449019; parent robot_base_link -> robot_chassis_link
- joint robot_sick_rear_supportsick_support_joint: origin xyz=-0.472 -0.3795 0.3774 rpy=0 1.57079632679 -1.57079632679 -> xyz=-0.472 -0.3795 0.09788 rpy=0 1.57079632679 -1.57079632679; parent robot_base_link -> robot_chassis_link

Commit message: Update rbvogui_xl_lift_ur10e.urdf

File: data/rbvogui_xl_lift_ur10e.urdf (robot description, URDF)
Before this commit: robot rbvogui, 39 links, 38 joints
Links:
- link robot_back_left_motor_wheel: geometry collision mesh filename=package://rbvogui_description/hub_rbvogui_xl.stl; visual mesh filename=package://rbvogui_description/hub_rbvogui_xl.stl
- link robot_back_left_wheel: geometry collision mesh filename=package://rbvogui_description/wheel_350mm.stl; visual mesh filename=package://rbvogui_description/wheel_350mm.stl
- link robot_back_right_motor_wheel: geometry collision mesh filename=package://rbvogui_description/hub_rbvogui_xl.stl; visual mesh filename=package://rbvogui_description/hub_rbvogui_xl.stl
- link robot_back_right_wheel: geometry collision mesh filename=package://rbvogui_description/wheel_350mm.stl; visual mesh filename=package://rbvogui_description/wheel_350mm.stl
- link robot_base_logos_link: geometry visual mesh filename=package://rbvogui_description/rbvogui_logos.stl scale=1.24 1.24 1
- link robot_battery_link: geometry collision mesh filename=package://rbvogui_description/rbvogui_xl_battery.stl; visual mesh filename=package://rbvogui_description/rbvogui_xl_battery.stl
- link robot_chassis_link: geometry collision mesh filename=package://rbvogui_description/rbvogui_xl_chassis.stl; visual mesh filename=package://rbvogui_description/rbvogui_xl_chassis.stl
- link robot_contactors_link: geometry visual mesh filename=package://rbvogui_description/rbvogui_contactors.stl
- link robot_ewellix_lift_base_link: geometry collision mesh filename=package://ewellix_description/ewellix_lift_base_700mm.stl; visual mesh filename=package://ewellix_description/ewellix_lift_base_700mm.stl
- link robot_ewellix_lift_top_link: geometry collision mesh filename=package://ewellix_description/ewellix_lift_top_700mm.stl; visual mesh filename=package://ewellix_description/ewellix_lift_top_700mm.stl
- link robot_front_3d_laser_base_link: geometry collision mesh filename=package://robotnik_sensors/rs_bpearl.stl; visual mesh filename=package://robotnik_sensors/rs_bpearl.stl
- link robot_front_left_motor_wheel: geometry collision mesh filename=package://rbvogui_description/hub_rbvogui_xl.stl; visual mesh filename=package://rbvogui_description/hub_rbvogui_xl.stl
- link robot_front_left_wheel: geometry collision mesh filename=package://rbvogui_description/wheel_350mm.stl; visual mesh filename=package://rbvogui_description/wheel_350mm.stl
- link robot_front_rgbd_camera_link: geometry collision mesh filename=package://robotnik_sensors/orbbec_astra.stl; visual mesh filename=package://robotnik_sensors/orbbec_astra.stl
- link robot_front_right_motor_wheel: geometry collision mesh filename=package://rbvogui_description/hub_rbvogui_xl.stl; visual mesh filename=package://rbvogui_description/hub_rbvogui_xl.stl
- link robot_front_right_wheel: geometry collision mesh filename=package://rbvogui_description/wheel_350mm.stl; visual mesh filename=package://rbvogui_description/wheel_350mm.stl
- link robot_gps_base_link: geometry collision mesh filename=package://robotnik_sensors/antenna_ANN_MB_mast.stl scale=1.0 1.0 1.0; visual mesh filename=package://robotnik_sensors/antenna_ANN_MB_mast.stl scale=1.0 1.0 1.0
- link robot_imu_base_link: geometry collision box size=0.036 0.037 0.009; visual mesh filename=package://robotnik_sensors/vectornav_vn100.stl
- link robot_leds_link: geometry visual mesh filename=package://rbvogui_description/rbvogui_xl_leds.stl
