Commit message: robotmodels update

File: data/rbvogui_xl_lift_ur10e_indoor.urdf (robot description, URDF)
Before this commit: robot rbvogui, 39 links, 38 joints
Links:
- link robot_back_left_wheel: geometry collision sphere radius=0.1425; visual mesh filename=package://rbvogui_description/meshes/wheels/wheel_285mm.stl
- link robot_back_right_wheel: geometry collision sphere radius=0.1425; visual mesh filename=package://rbvogui_description/meshes/wheels/wheel_285mm.stl
- link robot_front_left_wheel: geometry collision sphere radius=0.1425; visual mesh filename=package://rbvogui_description/meshes/wheels/wheel_285mm.stl
- link robot_front_right_wheel: geometry collision sphere radius=0.1425; visual mesh filename=package://rbvogui_description/meshes/wheels/wheel_285mm.stl
Joints:
- joint robot_arm_base_joint: origin xyz=0 0 0.015 rpy=0 0 2.35619449019 -> xyz=0 0 0.015 rpy=0 0 0.785398163397
- joint robot_arm_base_link-base_link_inertia: origin xyz=0 0 0 rpy=0 0 0 -> xyz=0 0 0 rpy=0 0 3.14159265359
- joint robot_base_footprint_joint: origin xyz=0 0 0.17 rpy=0 0 0 -> xyz=0 0 0.1425 rpy=0 0 0

Commit message: urdf fixes

File: data/rbvogui_xl_lift_ur10e_indoor.urdf (robot description, URDF)
Before this commit: robot rbvogui, 39 links, 38 joints
Joints:
- joint robot_arm_base_joint: origin xyz=0 0 0.015 rpy=0 0 0.785398163397 -> xyz=0 0 0.015 rpy=0 0 2.35619449019
- joint robot_arm_base_link-base_link_inertia: origin xyz=0 0 0 rpy=0 0 3.14159265359 -> xyz=0 0 0 rpy=0 0 0

Commit message: Correction of directories in indoor urdf

File: data/rbvogui_xl_lift_ur10e_indoor.urdf (robot description, URDF)
Before this commit: robot rbvogui, 39 links, 38 joints
Links:
- link robot_back_left_motor_wheel: geometry collision mesh filename=package://rbvogui_description/hub_rbvogui_xl.stl; visual mesh filename=package://rbvogui_description/hub_rbvogui_xl.stl
- link robot_back_left_wheel: geometry collision sphere radius=0.1425; visual mesh filename=package://rbvogui_description/wheel_285mm.stl
- link robot_back_right_motor_wheel: geometry collision mesh filename=package://rbvogui_description/hub_rbvogui_xl.stl; visual mesh filename=package://rbvogui_description/hub_rbvogui_xl.stl
- link robot_back_right_wheel: geometry collision sphere radius=0.1425; visual mesh filename=package://rbvogui_description/wheel_285mm.stl
- link robot_base_logos_link: geometry visual mesh filename=package://rbvogui_description/rbvogui_logos.stl scale=1.24 1.24 1
- link robot_battery_link: geometry collision mesh filename=package://rbvogui_description/rbvogui_xl_battery.stl; visual mesh filename=package://rbvogui_description/rbvogui_xl_battery.stl
- link robot_chassis_link: geometry collision mesh filename=package://rbvogui_description/rbvogui_xl_chassis.stl; visual mesh filename=package://rbvogui_description/rbvogui_xl_chassis.stl
- link robot_contactors_link: geometry visual mesh filename=package://rbvogui_description/rbvogui_contactors.stl
- link robot_ewellix_lift_base_link: geometry collision mesh filename=package://ewellix_description/ewellix_lift_base_700mm.stl; visual mesh filename=package://ewellix_description/ewellix_lift_base_700mm.stl
- link robot_ewellix_lift_top_link: geometry collision mesh filename=package://ewellix_description/ewellix_lift_top_700mm.stl; visual mesh filename=package://ewellix_description/ewellix_lift_top_700mm.stl
- link robot_front_left_motor_wheel: geometry collision mesh filename=package://rbvogui_description/hub_rbvogui_xl.stl; visual mesh filename=package://rbvogui_description/hub_rbvogui_xl.stl
- link robot_front_left_wheel: geometry collision sphere radius=0.1425; visual mesh filename=package://rbvogui_description/wheel_285mm.stl
- link robot_front_right_motor_wheel: geometry collision mesh filename=package://rbvogui_description/hub_rbvogui_xl.stl; visual mesh filename=package://rbvogui_description/hub_rbvogui_xl.stl
- link robot_front_right_wheel: geometry collision sphere radius=0.1425; visual mesh filename=package://rbvogui_description/wheel_285mm.stl
- link robot_leds_link: geometry visual mesh filename=package://rbvogui_description/rbvogui_xl_leds.stl

Commit message: Update rbvogui_xl_lift_ur10e_indoor.urdf

File: data/rbvogui_xl_lift_ur10e_indoor.urdf (robot description, URDF)
Before this commit: robot rbvogui, 39 links, 38 joints
Links:
- link robot_front_3d_laser_base_link: geometry collision mesh filename=package://robotnik_sensors/rs_bpearl.stl; visual mesh filename=package://robotnik_sensors/rs_bpearl.stl
- link robot_front_rgbd_camera_link: geometry collision mesh filename=package://robotnik_sensors/orbbec_astra.stl; visual mesh filename=package://robotnik_sensors/orbbec_astra.stl
- link robot_gps_base_link: geometry collision mesh filename=package://robotnik_sensors/antenna_ANN_MB_mast.stl scale=1.0 1.0 1.0; visual mesh filename=package://robotnik_sensors/antenna_ANN_MB_mast.stl scale=1.0 1.0 1.0
- link robot_imu_base_link: geometry collision box size=0.036 0.037 0.009; visual mesh filename=package://robotnik_sensors/vectornav_vn100.stl
