Commit message: Fix analytical inverse, added kinematics functions

File: data/robot_description/rbvogui_xl_ur20/rbvogui_xl_ur20.urdf (robot description, URDF)
Before this commit: robot rbvogui, 39 links, 38 joints
Joints:
- joint robot_arm_elbow_joint: limit lower=-3.141592653589793 upper=1.0 effort=430.0 velocity=2.6179938779914944 -> lower=-3.141592653589793 upper=3.141592653589793 effort=430.0 velocity=2.6179938779914944
